Commit message: Nove caster kolecka pro Lokiho + jednoduchý model kol pro Orphea

File: urdf/loki/loki_description (copy).urdf (robot description, URDF)
Before this commit: robot orpheus_x4, 4 links, 3 joints
Links:
- removed link platform_link
- added link front_caster; collision sphere radius=${(wheel_radius+wheel_zoff-(base_height/2))}; visual sphere radius=${(wheel_radius+wheel_zoff-(base_height/2))}
- added link rear_caster; collision sphere radius=${(wheel_radius+wheel_zoff-(base_height/2))}; visual sphere radius=${(wheel_radius+wheel_zoff-(base_height/2))}
- link base_link: geometry collision box size=${base_length} ${base_width} ${base_height}; visual mesh filename=file://$(find robot_models)/meshes/loki/Loki_base.stl scale=0.001 0.001 0.001
- link mounting_plate_link: geometry collision box size=${base_length} ${base_width} 0.001; visual mesh filename=file://$(find robot_models)/meshes/loki/Loki_mount_plate.stl scale=0.001 0.001 0.001
Joints:
- removed joint platform_joint
- added joint front_caster_joint: type fixed, parent base_link, child front_caster, origin xyz=${caster_xoff} 0.0 ${-(base_height/2)} rpy=0 0 0
- added joint rear_caster_joint: type fixed, parent base_link, child rear_caster, origin xyz=${-caster_xoff} 0.0 ${-(base_height/2)} rpy=0 0 0

File: urdf/loki/loki_description.urdf (robot description, URDF)
Before this commit: robot orpheus_x4, 5 links, 4 joints
Links:
- link base_link: geometry collision box size=${base_length} ${base_width} ${base_height}; visual mesh filename=file://$(find robot_models)/meshes/loki/Loki_base.stl scale=0.001 0.001 0.001
- link front_caster: geometry collision sphere radius=${(wheel_radius+wheel_zoff-(base_height/2))}; visual mesh filename=file://$(find robot_models)/meshes/loki/Loki_caster.stl scale=0.001 0.001 0.001
- link mounting_plate_link: geometry collision box size=${base_length} ${base_width} 0.001; visual mesh filename=file://$(find robot_models)/meshes/loki/Loki_mount_plate.stl scale=0.001 0.001 0.001
- link rear_caster: geometry collision sphere radius=${(wheel_radius+wheel_zoff-(base_height/2))}; visual mesh filename=file://$(find robot_models)/meshes/loki/Loki_caster.stl scale=0.001 0.001 0.001

File: urdf/orpheus_ac/orpheus_ac_description.urdf (robot description, URDF)
Before this commit: robot orpheus_ac, 4 links, 3 joints
Links:
- link Big_mounting_plate_link: geometry collision box size=${base_length} ${base_width} 0.001; visual mesh filename=file://$(find robot_models)/meshes/orpheus_ac/Mount_plate_o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 scale=0.001 0.001 0.001
- link Small_mounting_plate_link: geometry collision box size=${base_length} ${base_width} 0.001; visual mesh filename=file://$(find robot_models)/meshes/orpheus_ac/Mount_plate_o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 scale=0.001 0.001 0.001
- link base_link: geometry collision box size=${base_length} ${base_width} ${base_height}; visual mesh filename=file://$(find robot_models)/meshes/orpheus_ac/Base_orpheus_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 scale=0.001 0.001 0.001
