Commit message: Uprava barev a kolizniho modelu

File: urdf/orpheus_ac/orpheus_ac_description (copy).urdf (robot description, URDF)
Before this commit: robot orpheus_ac, 4 links, 3 joints
Links:
- link Big_mounting_plate_link: geometry collision box size=${base_length/1.8} ${base_width} 0.001; visual mesh filename=file://$(find robot_models)/meshes/orpheus_ac/Mount_plate_o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 scale=0.001 0.001 0.001
- link Small_mounting_plate_link: geometry collision box size=${base_length/3} ${base_width} 0.001; visual mesh filename=file://$(find robot_models)/meshes/orpheus_ac/Mount_plate_o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 scale=0.001 0.001 0.001
- link base_link: geometry collision box size=${base_length} ${base_width} ${base_height}; visual mesh filename=file://$(find robot_models)/meshes/orpheus_ac/Base_orpheus_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 scale=0.001 0.001 0.001
