Commit message: Uprava barev a pridani boxu na Orphea X4

File: urdf/orpheus_x4/orpheus_x4_description.urdf (robot description, URDF)
Before this commit: robot orpheus_x4, 4 links, 3 joints
Links:
- added link box_platform_link; collision box size=0.12 0.2 0.09; visual box size=0.12 0.2 0.09
Joints:
- added joint box_platform_joint: type fixed, parent platform_link, child box_platform_link, origin xyz=0.0 0.0 0.2325 rpy=0 0 0
